File: ISA_SerPaROM.sch (KiCad schematic (older format))
At the start: 70 parts, among them J1 ISA BUS, J10 Parallel Port, J2 ADDR_IRQ, J3 UART1_SEL, J4 UART2_SEL, J5 Parallel Port LEDs, J6 Serial 2 IDC, J7 Serial 1 DB9, J9 Parport IRQ Select, U1 74LS138, U11 74LS30, U12 74LS86, U13 74LS02, U14 74LS155, U15 74LS245, U16 74LS174, U17 74LS374, U18 74LS05, U19 74LS125, U2 74LS138, U20 74LS240, U21 74LS244, U22 16550, U4 16550, U5 GD75232N, U6 GD75232N, X1 1.8432Mhz

Commit message: Additional parallel ports
Parts:
- removed D1: LED RX1, LED_THT:LED_D3.0mm, symbol Device:LED_Small
- removed D2: LED TX1, LED_THT:LED_D3.0mm, symbol Device:LED_Small
- removed D3: LED RX2, LED_THT:LED_D3.0mm, symbol Device:LED_Small
- removed D4: LED TX2, LED_THT:LED_D3.0mm, symbol Device:LED_Small
- removed J5: Parallel Port LEDs, Package_DIP:DIP-20_W7.62mm_Socket_LongPads, symbol Connector_Generic:Conn_02x10_Counter_Clockwise
- removed R1, R2, R3, R4: 1k, Resistor_THT:R_Axial_DIN0207_L6.3mm_D2.5mm_P10.16mm_Horizontal, symbol Device:R_Small
- removed RN2: 1k, Resistor_THT:R_Array_SIP11, symbol Device:R_Network10
- removed U22, U4: 16550, Package_DIP:DIP-40_W15.24mm_LongPads, symbol Interface_UART:16550
- added C17, C18: 100nF, Capacitor_THT:C_Disc_D6.0mm_W2.5mm_P5.00mm, symbol Device:C_Small
- added J10: Serial 3 IDC, Connector_PinHeader_2.54mm:PinHeader_2x05_P2.54mm_Vertical, symbol Connector_Generic:Conn_02x05_Odd_Even
- added J11: Serial 4 IDC, Connector_PinHeader_2.54mm:PinHeader_2x05_P2.54mm_Vertical, symbol Connector_Generic:Conn_02x05_Odd_Even
- added J5: ADDR, Connector_PinHeader_2.54mm:PinHeader_1x04_P2.54mm_Vertical, symbol Connector_Generic:Conn_01x04
- added J8: UART3_SEL, Connector_PinHeader_2.54mm:PinHeader_1x04_P2.54mm_Vertical, symbol Connector_Generic:Conn_01x04
- added J9: UART4_SEL, Connector_PinHeader_2.54mm:PinHeader_1x04_P2.54mm_Vertical, symbol Connector_Generic:Conn_01x04
- added JP3: Interrupt Mode, Connector_PinHeader_2.54mm:PinHeader_1x02_P2.54mm_Vertical, symbol Device:Jumper_NO_Small
- added RN?: 4.7k, Resistor_THT:R_Array_SIP5, symbol Device:R_Network04
- added U23: 16C554, Package_LCC:PLCC-68_THT-Socket, symbol custom_components:16554
- added U24: 74LS32, Package_DIP:DIP-14_W7.62mm_LongPads, symbol 74xx:74LS32
- added U25, U26: GD75232N, Package_DIP:DIP-20_W7.62mm_LongPads, symbol Interface_UART:GD75232N
Connections:
- net labels added: RS232_3_CTS, RS232_3_DCD, RS232_3_DSR, RS232_3_DTR, RS232_3_RI, RS232_3_RTS, RS232_3_RX, RS232_3_TX, RS232_4_CTS, RS232_4_DCD, RS232_4_DSR, RS232_4_DTR, RS232_4_RI, RS232_4_RTS, RS232_4_RX, RS232_4_TX, RX_A, RX_B, RX_C, RX_D, TX_A, TX_B, TX_C, TX_D, UARTA_IRQ, UARTB_IRQ, UARTC_IRQ, UARTD_IRQ, ~CTS_A, ~CTS_B, ~CTS_C, ~CTS_D, ~DCD_A, ~DCD_B, ~DCD_C, ~DCD_D, ~DSR_A, ~DSR_B, ~DSR_C, ~DSR_D, ~DTR_A, ~DTR_B, ~DTR_C, ~DTR_D, ~RI_A, ~RI_B, ~RI_C, ~RI_D, ~RTS_A, ~RTS_B, ~RTS_C, ~RTS_D, ~UART3_CS, ~UART4_CS
- net labels removed: SIN_1, SIN_2, SOUT_1, SOUT_2, ~CTS_1, ~CTS_2, ~DCD_1, ~DCD_2, ~DSR_1, ~DSR_2, ~DTR_1, ~DTR_2, ~RI_1, ~RI_2, ~RTS_1, ~RTS_2
- wire segments 753 -> 810
- no-connect marks 42 -> 37
Other:
- moved on the sheet: J10, J2, J3, J4, J7, J9, U1, U12A, U12D, U13A, U18F, U19B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

Commit message: Route Serial/Parallel/ROM board
Parts:
- added C19, C20: 100nF, Capacitor_THT:C_Disc_D6.0mm_W2.5mm_P5.00mm, symbol Device:C_Small
- added D1: LED Channel A, LED_THT:LED_D3.0mm-3, symbol Device:LED_Dual_CAC
- added D2: LED Channel B, LED_THT:LED_D3.0mm-3, symbol Device:LED_Dual_CAC
- added D3: LED Channel C, LED_THT:LED_D3.0mm-3, symbol Device:LED_Dual_CAC
- added D4: LED Channel D, LED_THT:LED_D3.0mm-3, symbol Device:LED_Dual_CAC
- added J14: ROM Config, Connector_PinHeader_2.54mm:PinHeader_2x07_P2.54mm_Vertical, symbol Connector_Generic:Conn_02x07_Odd_Even
- added R1, R2: 10k, Resistor_THT:R_Axial_DIN0207_L6.3mm_D2.5mm_P10.16mm_Horizontal, symbol Device:R_Small
- added R10, R3, R4, R5, R6, R7, R8, R9: 1k, Resistor_THT:R_Axial_DIN0207_L6.3mm_D2.5mm_P10.16mm_Horizontal, symbol Device:R_Small
- added RN3: 10k, Resistor_THT:R_Array_SIP6, symbol Device:R_Network05
- added U27: SST39SF040, Package_DIP:DIP-32_W15.24mm_LongPads, symbol Memory_Flash:SST39SF040
- added U28: 74HCT688, Package_DIP:DIP-20_W7.62mm_LongPads, symbol 74xx:74HCT688
- gave numbers to parts that had none: 1
- renumbered J10 to J12, J9 to J13
Connections:
- net A0: now also U27.12 (A0)
- net A1: now also U27.11 (A1)
- net A10: now also U27.23 (A10)
- net A11: now also U27.25 (A11)
- net A12: now also U27.4 (A12)
- net A13: now also U27.28 (A13)
- net A14: now also U27.29 (A14)
- net A15: now also J14.1 (Pin_1), J14.3 (Pin_3)
- net A16: now also U28.11 (P4)
- net A17: now also U28.13 (P5)
- net A18: now also U28.15 (P6)
- net A19: now also U28.17 (P7)
- net A2: now also U27.10 (A2)
- net A3: now also U27.9 (A3)
- net A4: now also U27.8 (A4)
- net A5: now also U27.7 (A5)
- net A6: now also U27.6 (A6)
- net A7: now also U27.5 (A7)
- net A8: now also U27.27 (A8)
- net A9: now also U27.26 (A9)
- net D0: now also U27.13 (D0)
- net D1: now also U27.14 (D1)
- net D2: now also U27.15 (D2)
- net D3: now also U27.17 (D3)
- net D4: now also U27.18 (D4)
- net D5: now also U27.19 (D5)
- net D6: now also U27.20 (D6)
- net D7: now also U27.21 (D7)
- net GND: now also C19.2, C20.2, J14.11 (Pin_11), J14.13 (Pin_13), J14.5 (Pin_5), J14.7 (Pin_7), J14.9 (Pin_9), R1.1, R2.1, U27.1 (A18), U27.16 (GND), U27.2 (A16), U27.30 (A17), U28.10 (GND), U28.2 (P0), U28.3 (R0), U28.4 (P1), U28.5 (R1), U28.6 (P2), U28.7 (R2)
- net RX_A: now also R4.2
- net RX_B: now also R6.2
- net RX_C: now also R8.2
- net RX_D: now also R10.2
- net TX_A: now also R3.2
- net TX_B: now also R5.2
- net TX_C: now also R7.2
- net TX_D: now also R9.2
- net VCC: now also C19.1, C20.1, D1.2 (A), D2.2 (A), D3.2 (A), D4.2 (A), RN3.1 (common), U27.32 (VCC), U28.18 (R7), U28.20 (VCC)
- net ~MEMR: now also U27.24 (OE)
- net ~MEMW: now also U27.31 (PGM)
- new net: D1.1 (K1), R3.1
- new net: D1.3 (K2), R4.1
- new net: D2.1 (K1), R5.1
- new net: D2.3 (K2), R6.1
- new net: D3.1 (K1), R7.1
- new net: D3.3 (K2), R8.1
- new net: D4.1 (K1), R9.1
- new net: D4.3 (K2), R10.1
- new net COMPARATOR_A15: J14.2 (Pin_2), R1.2, U28.8 (P3)
- new net FLASH_A15: J14.4 (Pin_4), R2.2, U27.3 (A15)
- new net SW_A15: J14.12 (Pin_12), RN3.5 (R4), U28.9 (R3)
- new net SW_A16: J14.10 (Pin_10), RN3.4 (R3), U28.12 (R4)
- new net SW_A17: J14.8 (Pin_8), RN3.3 (R2), U28.14 (R5)
- new net SW_A18: J14.6 (Pin_6), RN3.2 (R1), U28.16 (R6)
- new net SW_ROM_EN: J14.14 (Pin_14), RN3.6 (R5), U28.1 (G)
- new net ~ROM-CS: U27.22 (CE), U28.19 (P=R)
Other:
- note added: "ROM"

Commit message: Add notes to the schematic, cleaned the silkscreen
Other:
- note added: "32K"
- note added: "32K ROM bank"
- note added: "64K"
- note added: "64K ROM bank"
- note added: "A000h"
- note added: "A15"
- note added: "A16"
- note added: "A17"
- note added: "A18"
- note added: "A800h"
- note added: "B000h"
- note added: "B800h"
- note added: "C000h"
- note added: "C800h"
- note added: "D000h"
- note added: "D800h"
- note added: "E000h"
- note added: "E800h"
- note added: "ENA"
- note added: "F000h"
- note added: "F800h"
- note added: "If 32K mode is set, the A15 line will\nnot be used to address the content\nof the ROM (FLASH_A15 will be always\nlow), but will be decoded by the\n'688 to decide whether the ROM gets\nenabled or not.\n\nIn 64K mode, the A15 line will be used\nto address the content of the ROM,\nthe A15 jumper MUST be set, otherwise\nthe decoder will fail to enable the ROM\n(note how the COMPARATOR_A15 line\nwill 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"
- note added: "Jumper ONE of these two to\nselect 32K or 64K ROM slot size"
- note added: "Jumper to ENABLE the ROM"
- note added: "Logic taken from https://www.lo-tech.co.uk/wiki/Lo-tech_ISA_ROM_Board"
- note added: "Remember that the comparator is\nhardwired to check for A19 to be HIGH!"
- note added: "X"
Changed lines of the file:
@@
 Text Label 22500 4900 2    50   ~ 0
 RX_D
+Text Notes 20750 9250 0    50   ~ 0
+32K
+Text Notes 20750 9350 0    50   ~ 0
+64K
+Text Notes 20750 9450 0    50   ~ 0
+A18
+Text Notes 20750 9550 0    50   ~ 0
+A17
+Text Notes 20750 9650 0    50   ~ 0
+A16
+Text Notes 20750 9750 0    50   ~ 0
+A15
+Text Notes 20750 9850 0    50   ~ 0
+ENA
+Wire Notes Line
+	20900 9200 21000 9200
+Wire Notes Line
+	21000 9200 21000 9300
+Wire Notes Line
+	21000 9300 20900 9300
+Text Notes 21050 9300 0    39   ~ 0
+Jumper ONE of these two to\nselect 32K or 64K ROM slot size
+Text Notes 21050 9850 0    39   ~ 0
+Jumper to ENABLE the ROM
+Wire Notes Line
+	20550 5900 20250 5900
+Wire Notes Line
+	20250 5900 20250 7300
+Wire Notes Line
+	20250 7300 20550 7300
+Text Notes 20250 6900 1    50   ~ 0
+32K ROM bank
+Wire Notes Line
+	20200 5900 20050 5900
+Wire Notes Line
+	20050 5900 20050 7400
+Wire Notes Line
+	20050 7400 20400 7400
+Text Notes 20050 6900 1    50   ~ 0
+64K ROM bank
+Text Notes 18700 7150 0    39   ~ 0
+If 32K mode is set, the A15 line will\nnot be used to address the content\nof the ROM (FLASH_A15 will be always\nlow), but will be decoded by the\n'688 to decide whether the ROM gets\nenabled or not.\n\nIn 64K mode, the A15 line will be used\nto address the content of the ROM,\nthe A15 jumper MUST be set, otherwise\nthe decoder will fail to enable the ROM\n(note how the COMPARATOR_A15 line\nwill be pulled low by R1).
+Text Notes 21750 10650 0    39   ~ 0
+A18
+Text Notes 21950 10650 0    39   ~ 0
+A17
+Text Notes 22150 10650 0    39   ~ 0
+A16
+Text Notes 22350 10650 0    39   ~ 0
+A15
+Wire Notes Line
+	22500 10700 21250 10700
+Wire Notes Line
+	21250 10850 22500 10850
+Text Notes 21350 10800 0    50   ~ 0
+A000h
+Wire Notes Line
+	21250 11000 22500 11000
+Wire Notes Line
+	21250 11150 22500 11150
+Wire Notes Line
+	21250 11300 22500 11300
+Wire Notes Line
+	21250 11450 22500 11450
+Wire Notes Line
+	21250 11600 22500 11600
+Wire Notes Line
+	22500 10600 22500 11600
+Wire Notes Line
+	21700 10600 21700 11600
+Wire Notes Line
+	21900 10600 21900 11600
+Wire Notes Line
+	22100 10600 22100 11600
+Wire Notes Line
+	22300 10600 22300 11600
+Text Notes 21350 10950 0    50   ~ 0
+B000h
+Text Notes 21350 11100 0    50   ~ 0
+C000h
+Text Notes 21350 11250 0    50   ~ 0
+D000h
+Text Notes 21350 11400 0    50   ~ 0
+E000h
+Text Notes 21350 11550 0    50   ~ 0
+F000h
+Text Notes 21350 10650 0    39   ~ 0
+64K
+Text Notes 22400 10800 0    50   ~ 0
+X
+Text Notes 22400 10950 0    50   ~ 0
+X
+Text Notes 22400 11100 0    50   ~ 0
+X
+Text Notes 22400 11250 0    50   ~ 0
+X
+Text Notes 22400 11400 0    50   ~ 0
+X
+Text Notes 22400 11550 0    50   ~ 0
+X
+Text Notes 22200 10800 0    50   ~ 0
+X
+Text Notes 21800 10800 0    50   ~ 0
+X
+Text Notes 21800 10950 0    50   ~ 0
+X
+Text Notes 22200 11100 0    50   ~ 0
+X
+Text Notes 22000 11100 0    50   ~ 0
+X
+Text Notes 22000 11250 0    50   ~ 0
+X
+Text Notes 22200 11400 0    50   ~ 0
+X
+Text Notes 21300 10500 0    39   ~ 0
+Remember that the comparator is\nhardwired to check for A19 to be HIGH!
+Text Notes 21750 11800 0    39   ~ 0
+A18
+Text Notes 21950 11800 0    39   ~ 0
+A17
+Text Notes 22150 11800 0    39   ~ 0
+A16
+Text Notes 22350 11800 0    39   ~ 0
+A15
+Wire Notes Line
+	22500 11850 21250 11850
+Wire Notes Line
+	21250 12000 22500 12000
+Text Notes 21350 11950 0    50   ~ 0
+A000h
+Wire Notes Line
+	21250 12150 22500 12150
+Wire Notes Line
+	21250 12300 22500 12300
+Wire Notes Line
+	21250 12450 22500 12450
+Wire Notes Line
+	21250 12600 22500 12600
+Wire Notes Line
+	21250 12750 22500 12750
+Text Notes 21350 12100 0    50   ~ 0
+A800h
+Text Notes 21350 12250 0    50   ~ 0
+B000h
+Text Notes 21350 12400 0    50   ~ 0
+B800h
+Text Notes 21350 12550 0    50   ~ 0
+C000h
+Text Notes 21350 12700 0    50   ~ 0
+C800h
+Text Notes 21350 11800 0    39   ~ 0
+32K
+Text Notes 22400 11950 0    50   ~ 0
+X
+Text Notes 22400 12250 0    50   ~ 0
+X
+Text Notes 22400 12550 0    50   ~ 0
+X
+Text Notes 22200 12700 0    50   ~ 0
+X
+Text Notes 22200 11950 0    50   ~ 0
+X
+Text Notes 21800 11950 0    50   ~ 0
+X
+Text Notes 21800 12100 0    50   ~ 0
+X
+Text Notes 21800 12250 0    50   ~ 0
+X
+Text Notes 21800 12400 0    50   ~ 0
+X
+Text Notes 22200 12550 0    50   ~ 0
+X
+Wire Notes Line
+	21250 12900 22500 12900
+Text Notes 21350 12850 0    50   ~ 0
+D000h
+Wire Notes Line
+	21250 13050 22500 13050
+Wire Notes Line
+	21250 13200 22500 13200
+Wire Notes Line
+	21250 13350 22500 13350
+Wire Notes Line
+	21250 13500 22500 13500
+Wire Notes Line
+	21250 13650 22500 13650
+Text Notes 21350 13000 0    50   ~ 0
+D800h
+Text Notes 21350 13150 0    50   ~ 0
+E000h
+Text Notes 21350 13300 0    50   ~ 0
+E800h
+Text Notes 21350 13450 0    50   ~ 0
+F000h
+Text Notes 21350 13600 0    50   ~ 0
+F800h
+Text Notes 22400 12850 0    50   ~ 0
+X
+Text Notes 22400 13150 0    50   ~ 0
+X
+Text Notes 22400 13450 0    50   ~ 0
+X
+Text Notes 22000 12850 0    50   ~ 0
+X
+Text Notes 22200 13150 0    50   ~ 0
+X
+Text Notes 22200 13300 0    50   ~ 0
+X
+Wire Notes Line
+	22500 11750 22500 13650
+Wire Notes Line
+	21700 11750 21700 13650
+Wire Notes Line
+	21900 11750 21900 13650
+Wire Notes Line
+	22100 11750 22100 13650
+Wire Notes Line
+	22300 11750 22300 13650
+Text Notes 22200 12100 0    50   ~ 0
+X
+Text Notes 22000 12550 0    50   ~ 0
+X
+Text Notes 22000 12700 0    50   ~ 0
+X
+Text Notes 22000 13000 0    50   ~ 0
+X
 Wire Bus Line
 	13800 7800 13800 13500
@@
 Wire Bus Line
 	7650 9100 7650 13500
+Text Notes 18700 14650 0    39   ~ 0
+Logic taken from https://www.lo-tech.co.uk/wiki/Lo-tech_ISA_ROM_Board
 $EndSCHEMATC

Commit message: Update silkscreen
Parts:
- RN2: value 4.7k -> 10k
- U1, U2: value 74LS138 -> 74HCT138
- U24: value 74LS32 -> 74HCT32
Changed lines of the file:
@@
 Title "Serial + Parallel + ROM ISA Adapter"
 Date ""
-Rev "1.0"
+Rev "1.1"
 Comp ""
 Comment1 ""
@@
 P 14550 3550
 F 0 "U2" H 14300 4000 50  0000 C CNN
-F 1 "74LS138" H 14750 4000 50  0000 C CNN
+F 1 "74HCT138" H 14750 4000 50  0000 C CNN
 F 2 "Package_DIP:DIP-16_W7.62mm_LongPads" H 14550 3550 50  0001 C CNN
 F 3 "http://www.ti.com/lit/gpn/sn74LS138" H 14550 3550 50  0001 C CNN
@@
 P 14550 1700
 F 0 "U1" H 14300 2150 50  0000 C CNN
-F 1 "74LS138" H 14750 2150 50  0000 C CNN
+F 1 "74HCT138" H 14750 2150 50  0000 C CNN
 F 2 "Package_DIP:DIP-16_W7.62mm_LongPads" H 14550 1700 50  0001 C CNN
 F 3 "http://www.ti.com/lit/gpn/sn74LS138" H 14550 1700 50  0001 C CNN
@@
 P 1750 2550
 F 0 "U24" H 1750 2875 50  0000 C CNN
-F 1 "74LS32" H 1750 2784 50  0000 C CNN
+F 1 "74HCT32" H 1750 2784 50  0000 C CNN
 F 2 "Package_DIP:DIP-14_W7.62mm_LongPads" H 1750 2550 50  0001 C CNN
 F 3 "http://www.ti.com/lit/gpn/sn74LS32" H 1750 2550 50  0001 C CNN
@@
 P 1750 3100
 F 0 "U24" H 1750 3425 50  0000 C CNN
-F 1 "74LS32" H 1750 3334 50  0000 C CNN
+F 1 "74HCT32" H 1750 3334 50  0000 C CNN
 F 2 "" H 1750 3100 50  0001 C CNN
 F 3 "http://www.ti.com/lit/gpn/sn74LS32" H 1750 3100 50  0001 C CNN
@@
 P 1750 3650
 F 0 "U24" H 1750 3975 50  0000 C CNN
-F 1 "74LS32" H 1750 3884 50  0000 C CNN
+F 1 "74HCT32" H 1750 3884 50  0000 C CNN
 F 2 "" H 1750 3650 50  0001 C CNN
 F 3 "http://www.ti.com/lit/gpn/sn74LS32" H 1750 3650 50  0001 C CNN
@@
 P 1750 4200
 F 0 "U24" H 1750 4525 50  0000 C CNN
-F 1 "74LS32" H 1750 4434 50  0000 C CNN
+F 1 "74HCT32" H 1750 4434 50  0000 C CNN
 F 2 "" H 1750 4200 50  0001 C CNN
 F 3 "http://www.ti.com/lit/gpn/sn74LS32" H 1750 4200 50  0001 C CNN
@@
 P 3150 3900
 F 0 "U24" H 3380 3946 50  0000 L CNN
-F 1 "74LS32" H 3380 3855 50  0000 L CNN
+F 1 "74HCT32" H 3380 3855 50  0000 L CNN
 F 2 "" H 3150 3900 50  0001 C CNN
 F 3 "http://www.ti.com/lit/gpn/sn74LS32" H 3150 3900 50  0001 C CNN
@@
 P 3900 2050
 F 0 "RN2" H 3450 2150 50  0000 L CNN
-F 1 "4.7k" H 3600 2000 50  0000 R CNN
+F 1 "10k" H 3600 2000 50  0000 R CNN
 F 2 "Resistor_THT:R_Array_SIP5" V 4175 2050 50  0001 C CNN
 F 3 "http://www.vishay.com/docs/31509/csc.pdf" H 3900 2050 50  0001 C CNN
@@
 Text Notes 22000 13000 0    50   ~ 0
 X
+Text Notes 18700 14650 0    39   ~ 0
+Logic taken from https://www.lo-tech.co.uk/wiki/Lo-tech_ISA_ROM_Board
 Wire Bus Line
 	13800 7800 13800 13500
@@
 Wire Bus Line
 	7650 9100 7650 13500
-Text Notes 18700 14650 0    39   ~ 0
-Logic taken from https://www.lo-tech.co.uk/wiki/Lo-tech_ISA_ROM_Board
 $EndSCHEMATC
