File: ISA_SerPaROM.kicad_pcb (KiCad board)
At the start: 2 copper layers, 158.8 x 102.9 mm, 77 parts, among them J1 ISA BUS, J10 Parallel Port, J11 Serial 4 IDC, J12 Serial 3 IDC, J13 UART4_SEL, J2 ADDR_IRQ, J3 UART1_SEL, J4 UART2_SEL, J5 ADDR, J6 Serial 2 IDC, J7 Serial 1 DB9, J8 UART3_SEL, J9 Parport IRQ Select, U1 74HCT138, U11 74LS30, U12 74LS86, U13 74LS02, U14 74LS155, U15 74LS245, U16 74LS174, U17 74LS374, U18 74LS05, U19 74LS125, U2 74HCT138, U20 74LS240, U21 74LS244, U23 16C554, U24 74HCT32, U25 GD75232N, U26 GD75232N, U29 74HCT245, U30 74HCT21, U5 GD75232N, U6 GD75232N, X1 1.8432Mhz

Commit message: Updated silkscreen, again
Other:
- board text added: "9x 2.2nF"
- board text removed: "<- 9x 2.2nF ->"
Changed lines of the file:
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@@
   (general
     (thickness 1.6)
-    (drawings 68)
+    (drawings 71)
     (tracks 2785)
     (zones 0)
@@
     (descr "5-pin Resistor SIP pack")
     (tags R)
-    (fp_text reference RN2 (at 0 -2.4 90) (layer F.SilkS)
+    (fp_text reference RN2 (at -3.556 0.127 90) (layer F.SilkS)
       (effects (font (size 1 1) (thickness 0.15)))
     )
@@
     )
   )
+  (gr_line (start 214.63 120.015) (end 214.63 119.38) (layer F.SilkS) (width 0.12))
+  (gr_line (start 184.15 120.015) (end 184.15 119.38) (layer F.SilkS) (width 0.12))
+  (gr_line (start 184.15 120.015) (end 214.63 120.015) (layer F.SilkS) (width 0.12))
   (gr_text 74HCT21 (at 269.494 182.372 -90) (layer F.SilkS)
     (effects (font (size 1 1) (thickness 0.15)))
@@
     (effects (font (size 0.8 0.8) (thickness 0.15)))
   )
-  (gr_text "<- 9x 2.2nF ->" (at 194.31 120.65) (layer F.SilkS)
+  (gr_text "9x 2.2nF" (at 194.945 120.65) (layer F.SilkS)
     (effects (font (size 0.8 0.8) (thickness 0.15)) (justify left))
   )
